Commit message: Fixed typo

File: vehicle_simulation/air_description/urdf/sensors/VLP-16.urdf.xacro (robot description, xacro)
@@ -24,5 +24,5 @@
             <visual>
                 <geometry>
-                    <mesh filename="file:///$(find air_description)meshes/VLP16_base_2.dae" />
+                    <mesh filename="file:///$(find air_description)/meshes/VLP16_base_2.dae" />
                     <!-- <mesh filename="file:///$(find air_description)/models/twizy/meshes/VLP16_base_2.dae" /> -->
                 </geometry>
