Commit message: Added footprint_link and base_to_footprint joint

File: vehicle_simulation/air_description/urdf/bases/sd_twizy_body.urdf.xacro (robot description, xacro)
@@ -22,4 +22,13 @@
       </visual>
     </link>
+  <!-- Define the footprint_link -->
+  <link name="footprint_link">
+  </link>
+  <!-- Connect the footprint_link to the base_link (or whatever your main link is) -->
+  <joint name="base_to_footprint" type="fixed">
+    <parent link="base_link"/>
+    <child link="footprint_link"/>
+    <origin xyz="0 0 0" rpy="0 0 0"/>
+  </joint>
     <joint name="chassis_joint" type="fixed">
       <origin xyz="${wheelbase / 2} 0 0" rpy="0 0 0"/>

Commit message: Teleoperation Done: Fixed load of vehicle_control plugin
Main fixes: Joints and its links

File: vehicle_simulation/air_description/urdf/bases/sd_twizy_body.urdf.xacro (robot description, xacro)
@@ -29,5 +29,5 @@
     <parent link="base_link"/>
     <child link="footprint_link"/>
-    <origin xyz="0 0 0" rpy="0 0 0"/>
+    <origin xyz="${wheelbase} 0 ${clearance}" rpy="0 0 0"/>
   </joint>
     <joint name="chassis_joint" type="fixed">

File: vehicle_simulation/air_description/urdf/sd_twizy.urdf.xacro (robot description, xacro)
@@ -62,5 +62,5 @@
   <gazebo>
     <plugin name="vehicle_control" filename="libvehicle_control.so">
-      <!-- <ros>
+      <ros>
         <namespace>/sd_twizy</namespace>
       </ros>
@@ -72,11 +72,18 @@
       <jointName>rear_right_wheel_joint</jointName>
       <updateRate>100.0</updateRate>
-      <alwaysOn>true</alwaysOn> -->
+      <alwaysOn>true</alwaysOn>
     </plugin>
   </gazebo>
   <gazebo>
     <plugin name="joint_state_publisher" filename="libgazebo_ros_joint_state_publisher.so">
-      <robotNamespace>/sd_twizy</robotNamespace>
-      <jointName>front_left_wheel_joint, front_right_wheel_joint, front_left_steer_joint, front_right_steer_joint, rear_left_wheel_joint, rear_right_wheel_joint </jointName>
+      <ros>
+        <namespace>/sd_twizy</namespace>
+      </ros>
+      <jointName>front_left_wheel_joint</jointName>
+      <jointName>front_right_wheel_joint</jointName>
+      <jointName>front_left_steer_joint</jointName>
+      <jointName>front_right_steer_joint</jointName>
+      <jointName>rear_left_wheel_joint</jointName>
+      <jointName>rear_right_wheel_joint</jointName>
       <updateRate>100.0</updateRate>
       <alwaysOn>true</alwaysOn>

File: vehicle_simulation/air_description/urdf/wheels/sd_twizy_suspension.urdf.xacro (robot description, xacro)
@@ -141,5 +141,5 @@
   </link>
   <xacro:macro name="FL_wheel">
-    <joint name="front_left_steer_joint" type="fixed">
+    <joint name="front_left_steer_joint" type="revolute">
       <parent link="base_link"/>
       <child link="front_left_axle"/>
@@ -148,13 +148,14 @@
       <limit lower="-0.785398" upper="0.785398" effort="500000" velocity="250"/>
     </joint>
-    <joint name="front_left_wheel_joint" type="fixed">
+    <joint name="front_left_wheel_joint" type="revolute">
       <parent link="front_left_axle"/>
       <child link="front_left_wheel"/>
       <origin xyz="0 0 0" rpy="0 0 0"/>
       <axis xyz="0 0 -1"/>
+      <limit lower="-1e9" upper="1e9" effort="1000" velocity="1000"/>
     </joint>
   </xacro:macro>
   <xacro:macro name="FR_wheel">
-    <joint name="front_right_steer_joint" type="fixed">
+    <joint name="front_right_steer_joint" type="revolute">
       <parent link="base_link"/>
       <child link="front_right_axle"/>
@@ -163,25 +164,28 @@
       <limit lower="-0.785398" upper="0.785398" effort="500000" velocity="250"/>
     </joint>
-    <joint name="front_right_wheel_joint" type="fixed">
+    <joint name="front_right_wheel_joint" type="revolute">
       <parent link="front_right_axle"/>
       <child link="front_right_wheel"/>
       <origin xyz="0 0 0" rpy="0 0 0"/>
       <axis xyz="0 0 -1"/>
+      <limit lower="-1e9" upper="1e9" effort="1000" velocity="1000"/>
     </joint>
   </xacro:macro>
   <xacro:macro name="RL_wheel">
-    <joint name="rear_left_wheel_joint" type="fixed">
+    <joint name="rear_left_wheel_joint" type="revolute">
       <parent link="base_link"/>
       <child link="rear_left_wheel"/>
       <origin xyz="0 ${-(track / 2)} 0" rpy="${degrees_90} 0 0"/>
       <axis xyz="0 0 -1"/>
+      <limit lower="-1e9" upper="1e9" effort="1000" velocity="1000"/>
     </joint>
   </xacro:macro>
   <xacro:macro name="RR_wheel">
-    <joint name="rear_right_wheel_joint" type="fixed">
+    <joint name="rear_right_wheel_joint" type="revolute">
       <parent link="base_link"/>
       <child link="rear_right_wheel"/>
       <origin xyz="0 ${(track / 2)} 0" rpy="${degrees_90} 0 0"/>
       <axis xyz="0 0 -1"/>
+      <limit lower="-1e9" upper="1e9" effort="1000" velocity="1000"/>
     </joint>
   </xacro:macro>
