Commit message: Fixed colors and materials typos in car description xacro files

File: vehicle_simulation/air_description/urdf/bases/sd_twizy_body.gazebo.xacro (robot description, xacro)
@@ -7,5 +7,5 @@
 <robot xmlns:xacro="http://www.ros.org/wiki/xacro">
   <gazebo reference="chassis">
-    <material>Gazebo/Green</material>
+    <material>Gazebo/Blue</material>
   </gazebo>
 </robot>

File: vehicle_simulation/air_description/urdf/sensors/cameras.urdf.xacro (robot description, xacro)
@@ -26,5 +26,7 @@
           <box size="0.026 0.026 0.0203"/>
         </geometry>
-        <material name="red"/>
+        <material name="red">
+          <color rgba="1.0 0.0 0.0 1.0"/>
+        </material>
       </visual>
       <inertial>

File: vehicle_simulation/air_description/urdf/wheels/sd_twizy_suspension.urdf.xacro (robot description, xacro)
@@ -77,5 +77,7 @@
         <cylinder radius="${front_tyre_radius}" length="${front_tyre_width}"/>
       </geometry>
-      <material name="tire_mat"/>
+      <material name="tire_mat">
+        <color rgba="0.1 0.1 0.1 1.0"/>
+      </material>
     </visual>
   </link>
@@ -97,5 +99,7 @@
         <cylinder radius="${front_tyre_radius}" length="${front_tyre_width}"/>
       </geometry>
-      <material name="tire_mat"/>
+      <material name="tire_mat">
+        <color rgba="0.1 0.1 0.1 1.0"/>
+      </material>
     </visual>
   </link>
@@ -117,5 +121,7 @@
         <cylinder radius="${rear_tyre_radius}" length="${rear_tyre_width}"/>
       </geometry>
-      <material name="tire_mat"/>
+      <material name="tire_mat">
+        <color rgba="0.1 0.1 0.1 1.0"/>
+      </material>
     </visual>
   </link>
@@ -137,5 +143,7 @@
         <cylinder radius="${rear_tyre_radius}" length="${rear_tyre_width}"/>
       </geometry>
-      <material name="tire_mat"/>
+      <material name="tire_mat">
+        <color rgba="0.1 0.1 0.1 1.0"/>
+      </material>
     </visual>
   </link>
