Commit message: fix(air_description): adjust urdf files to proper vlp-16 usage

File: vehicle_simulation/air_description/urdf/sd_twizy.urdf.xacro (robot description, xacro)
@@ -11,5 +11,4 @@
   <xacro:include filename="$(find air_description)/urdf/bases/sd_twizy_body.urdf.xacro" />
   <xacro:include filename="$(find air_description)/urdf/wheels/sd_twizy_suspension.urdf.xacro" />
-  <xacro:include filename="$(find air_description)/urdf/sensors/VLP-16.urdf.xacro"/>
   <xacro:include filename="$(find air_description)/urdf/sensors/cameras.urdf.xacro"/>
   <xacro:arg name="pub_tf" default="true" />
@@ -22,6 +21,11 @@
   <xacro:FL_wheel/>
   <xacro:FR_wheel/>
+  <xacro:arg name="gpu" default="false"/>
+  <xacro:property name="gpu" value="$(arg gpu)" />
+  <xacro:arg name="organize_cloud" default="false"/>
+  <xacro:property name="organize_cloud" value="$(arg organize_cloud)" />
   <!-- Sensors -->
-  <xacro:VLP-16  parent="chassis" name="velodyne" topic="/points_raw" hz="10" samples="1875">
+  <xacro:include filename="$(find velodyne_description)/urdf/VLP-16.urdf.xacro"/>
+  <xacro:VLP-16 parent="base_link" name="velodyne" topic="/velodyne_points" organize_cloud="${organize_cloud}" hz="5" samples="440" gpu="${gpu}">
     <origin xyz="-0.681 0 1.445" rpy="0 -${1.5*M_PI/180.0} 0"/>
   </xacro:VLP-16>
